File: pcb/ik_dragonfly.brd (EAGLE design)
At the start: 41.1 x 20.3 mm, 32 parts, among them IC1 FT230X, IC2 ATXMEGA32E5, J1 2X03, U1 MIC5219-3.3, U2 LM4040

Commit message: updated BOM
Parts:
- IC1: value FT230X -> ATXMEGA32E5; device Ai_IC:SSOP-16-FTDI -> Ai_IC:TQFP32-08
- IC2: value ATXMEGA32E5 -> FT230X; device Ai_IC:TQFP32-08 -> Ai_IC:SSOP-16-FTDI
- L: value (none) -> YELLOW
- L1, L2: value (none) -> 33@100MHz
- ON: value (none) -> BLUE
- R1, R2: value (none) -> 22
- R3, R6: value (none) -> 1K
- R4: value (none) -> 330
- moved IC1 11.7 mm to (22.4, 10.3)
- moved IC2 11.7 mm to (10.8, 9.02)
- moved U$3 3.66 mm to (18.2, 4.19), turned to 90 degrees
- renumbered LED1 to ON, LED2 to L
Connections:
- net !RTS: now also IC2.2; no longer IC1.2
- net 3V3: now also IC1.17; no longer IC2.17
- net 5V: now also IC2.12; no longer IC1.12
- net AVCC: now also IC1.32; no longer IC2.32
- net D+: now also IC2.8; no longer IC1.8
- net D-: now also IC2.9; no longer IC1.9
- net FT_3V3: now also IC2.10, IC2.11, IC2.3; no longer IC1.10, IC1.11, IC1.3
- net FT_RX: now also IC1.21, IC2.4; no longer IC1.4, IC2.21
- net FT_TX: now also IC1.22, IC2.1; no longer IC1.1, IC2.22
- net GND: now also IC1.1, IC1.18, IC2.13, IC2.5; no longer IC1.13, IC1.5, IC2.1, IC2.18
- net PA0: now also IC1.6; no longer IC2.6
- net PA1: now also IC1.5; no longer IC2.5
- net PA2: now also IC1.4; no longer IC2.4
- net PA3: now also IC1.3; no longer IC2.3
- net PA4: now also IC1.2; no longer IC2.2
- net PA5: now also IC1.31; no longer IC2.31
- net PA6: now also IC1.30; no longer IC2.30
- net PA7: now also IC1.29; no longer IC2.29
- net PC0: now also IC1.16; no longer IC2.16
- net PC1: now also IC1.15; no longer IC2.15
- net PC2: now also IC1.14; no longer IC2.14
- net PC3: now also IC1.13; no longer IC2.13
- net PC4: now also IC1.12; no longer IC2.12
- net PC5: now also IC1.11; no longer IC2.11
- net PC6: now also IC1.10; no longer IC2.10
- net PC7: now also IC1.9; no longer IC2.9
- net PD0: now also IC1.28; no longer IC2.28
- net PD1: now also IC1.27; no longer IC2.27
- net PD2: now also IC1.26; no longer IC2.26
- net PD3: now also IC1.25; no longer IC2.25
- net PD4: now also IC1.24; no longer IC2.24
- net PD5: now also IC1.23; no longer IC2.23
- net PDI_C: now also IC1.8; no longer IC2.8
- net PDI_D: now also IC1.7; no longer IC2.7
- net PR0: now also IC1.20; no longer IC2.20
- net PR1: now also IC1.19; no longer IC2.19
Other:
- board text added: "DRAGONFLY"
- board text removed: "XmegaE5 Dev"

Commit message: finished BOM
Parts:
- removed R7: (no value), Ai_Passives:RES-0603
- added R5: 1K, Ai_Passives:RES-0603
- R3: value 1K -> 10K
- R4: value 330 -> 300
- moved R6 12.9 mm to (28.4, 12.3), turned to 90 degrees
Connections:
- net 3V3: now also R5.1; no longer R6.1
- net N$8: now also R5.2; no longer R6.2
- net N$9: now also R6.2; no longer R7.2
- net PA0: now also R6.1; no longer R7.1
Changed lines of the file:
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@@
 <element name="J1" library="Ai_Connectors" package="2X03" value="2X03" x="38.1" y="10.16" smashed="yes" rot="R270"/>
 <element name="U1" library="Ai_Power" package="SOT23-5" value="MIC5219-3.3" x="10.6299" y="15.39875" smashed="yes" rot="R270"/>
-<element name="R4" library="Ai_Passives" package="RES-0603" value="330" x="38.1" y="15.367" smashed="yes" rot="R180">
+<element name="R4" library="Ai_Passives" package="RES-0603" value="300" x="38.1" y="15.367" smashed="yes" rot="R180">
 <attribute name="NAME" x="37.6555" y="14.19225" size="0.6096" layer="25" font="vector" ratio="15"/>
 </element>
@@
 <attribute name="NAME" x="31.97225" y="11.96975" size="0.6096" layer="25" font="vector" ratio="15"/>
 </element>
-<element name="R3" library="Ai_Passives" package="RES-0603" value="1K" x="37.592" y="5.207" smashed="yes">
+<element name="R3" library="Ai_Passives" package="RES-0603" value="10K" x="37.592" y="5.207" smashed="yes">
 <attribute name="NAME" x="39.1795" y="5.04825" size="0.6096" layer="25" font="vector" ratio="15"/>
 </element>
@@
 <attribute name="NAME" x="19.05" y="16.03375" size="0.6096" layer="25" font="vector" ratio="15"/>
 </element>
-<element name="R6" library="Ai_Passives" package="RES-0603" value="1K" x="16.1925" y="16.1925" smashed="yes">
+<element name="R5" library="Ai_Passives" package="RES-0603" value="1K" x="16.1925" y="16.1925" smashed="yes">
 <attribute name="NAME" x="16.8275" y="15.39875" size="0.6096" layer="25" font="vector" ratio="15" rot="R180"/>
 </element>
 <element name="ON" library="Ai_LED" package="LED-0603" value="BLUE" x="16.35125" y="14.12875" smashed="yes" rot="R90"/>
 <element name="LOGO1" library="SparkFun-Aesthetics" package="OSHW-LOGO-S" value="OSHW-LOGOS" x="22.352" y="13.208" smashed="yes" rot="MR0"/>
-<element name="R7" library="Ai_Passives" package="RES-0603" value="" x="28.448" y="12.319" smashed="yes" rot="R90">
+<element name="R6" library="Ai_Passives" package="RES-0603" value="1K" x="28.448" y="12.319" smashed="yes" rot="R90">
 <attribute name="NAME" x="28.12415" y="10.02665" size="0.6096" layer="25" font="vector" ratio="15" rot="R90"/>
 <attribute name="VALUE" x="30.353" y="11.684" size="1.27" layer="27" rot="R90"/>
@@
 <signal name="PA0">
 <contactref element="IC1" pad="6"/>
-<contactref element="R7" pad="1"/>
+<contactref element="R6" pad="1"/>
 <contactref element="U2" pad="1"/>
 <wire x1="26.67635" y1="11.51875" x2="28.4025" y2="11.51875" width="0.254" layer="1"/>
@@
 <contactref element="R3" pad="2"/>
 <contactref element="C8" pad="1"/>
-<contactref element="R6" pad="1"/>
+<contactref element="R5" pad="1"/>
 <contactref element="L2" pad="2"/>
 <wire x1="11.90625" y1="16.37885" x2="11.93" y2="16.34875" width="0.254" layer="1"/>
@@
 <signal name="N$8">
 <contactref element="ON" pad="A"/>
-<contactref element="R6" pad="2"/>
+<contactref element="R5" pad="2"/>
 <wire x1="17.10125" y1="14.12875" x2="17.10125" y2="16.13375" width="0.254" layer="1"/>
 <wire x1="17.10125" y1="16.13375" x2="17.0925" y2="16.1925" width="0.254" layer="1"/>
 </signal>
 <signal name="N$9">
-<contactref element="R7" pad="2"/>
+<contactref element="R6" pad="2"/>
 <contactref element="L2" pad="1"/>
 <contactref element="C6" pad="1"/>

Commit message: finished (for reals) BOM
Parts:
- RST: device Ai_Electromechanical:SW-SPST-SMD03X026 -> Ai_Electromechanical:SW-SPST-SMD035X030
- moved RST 0.77 mm to (32.7, 7.02)
- moved L1 0.38 mm to (28.2, 6.19)
- moved R3 0.13 mm to (37.7, 5.21)
Routing:
- net 3V3: track 66.4 -> 64.9 mm
- net GND: vias 23 -> 22

Commit message: minor revision
Parts:
- LOGO1: device SparkFun-Aesthetics:OSHW-LOGO-S -> Ai_Miscellany:OSHW-LOGO-S
- RST: value SW-SPSTSMD03X026 -> SW-SPSTSMD035X030
Other:
- board text added: "By Ihsan Kehribar"
- board text removed: "Ihsan Kehribar"
Changed lines of the file:
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@@
 <setting verticaltext="up"/>
 </settings>
-<grid distance="5" unitdist="mil" unit="mil" style="lines" multiple="1" display="yes" altdistance="0.025" altunitdist="inch" altunit="inch"/>
+<grid distance="0.05" unitdist="inch" unit="inch" style="lines" multiple="1" display="yes" altdistance="0.025" altunitdist="inch" altunit="inch"/>
 <layers>
 <layer number="1" name="Top" color="4" fill="1" visible="yes" active="yes"/>
@@
 <wire x1="11.90625" y1="17.93875" x2="11.90625" y2="17.30375" width="0.1905" layer="21"/>
 <wire x1="11.7475" y1="17.30375" x2="11.90625" y2="17.30375" width="0.1905" layer="21"/>
-<text x="29.4005" y="15.60195" size="1.524" layer="22" ratio="15" rot="MR0">ATxmega32E5</text>
 <dimension x1="41.148" y1="20.32" x2="0" y2="20.32" x3="20.574" y3="22.06625" textsize="1.778" textratio="15" layer="49"/>
-<text x="15.367" y="7.20725" size="1.016" layer="22" font="vector" ratio="15" rot="MR180">Ihsan Kehribar</text>
-<text x="14.224" y="5.55625" size="1.016" layer="22" font="vector" ratio="15" rot="MR180">www.acrobotic.com</text>
+<text x="16.129" y="6.44525" size="0.8128" layer="22" font="vector" ratio="15" rot="MR180">By Ihsan Kehribar</text>
+<text x="16.51" y="5.04825" size="0.8128" layer="22" font="vector" ratio="15" rot="MR180">www.acrobotic.com</text>
 <text x="40.90035" y="16.3322" size="0.6096" layer="21" font="vector" ratio="15" rot="R90">v1.0</text>
 <text x="17.272" y="6.985" size="0.8128" layer="21" font="vector" ratio="15" rot="R90">DRAGONFLY</text>
+<text x="27.8765" y="16.61795" size="1.27" layer="22" ratio="15" rot="MR0">DRAGONFLY</text>
+<text x="26.6065" y="15.34795" size="0.8128" layer="22" ratio="15" rot="MR0">ATxmega32E5</text>
 </plain>
 <attributes>
@@
 </element>
 <element name="ON" library="Ai_LED" package="LED-0603" value="BLUE" x="16.35125" y="14.12875" smashed="yes" rot="R90"/>
-<element name="LOGO1" library="SparkFun-Aesthetics" package="OSHW-LOGO-S" value="OSHW-LOGOS" x="22.352" y="13.208" smashed="yes" rot="MR0"/>
+<element name="LOGO1" library="Ai_Miscellany" package="OSHW-LOGO-S" value="OSHW-LOGOS" x="22.352" y="13.208" smashed="yes" rot="MR0"/>
 <element name="R6" library="Ai_Passives" package="RES-0603" value="1K" x="28.448" y="12.319" smashed="yes" rot="R90">
 <attribute name="NAME" x="28.12415" y="10.02665" size="0.6096" layer="25" font="vector" ratio="15" rot="R90"/>
@@
 </element>
 <element name="USB1" library="Ai_Connectors" package="USB-MICROB-TH" value="USBMICROB-TH" x="1.74625" y="10.16" smashed="yes" rot="R270"/>
-<element name="RST" library="Ai_Electromechanical" package="SW-SPST-SMD035X030" value="SW-SPSTSMD03X026" x="32.7025" y="7.01675" smashed="yes" rot="R180">
+<element name="RST" library="Ai_Electromechanical" package="SW-SPST-SMD035X030" value="SW-SPSTSMD035X030" x="32.7025" y="7.01675" smashed="yes" rot="R180">
 <attribute name="NAME" x="34.163" y="4.953" size="0.6096" layer="21" font="vector" ratio="15"/>
 </element>
