File: pcb/ik_dragonfly.sch (EAGLE design)
At the start: 32 parts, among them IC1 FT230X, IC2 ATXMEGA32E5, J1 2X03, U1 MIC5219-3.3, U2 LM4040

Commit message: updated BOM
Parts:
- IC1: value FT230X -> ATXMEGA32E5; device Ai_IC:FT230X -> Ai_IC:ATXMEGA32E5
- IC2: value ATXMEGA32E5 -> FT230X; device Ai_IC:ATXMEGA32E5 -> Ai_IC:FT230X
- L: value (none) -> YELLOW
- L1, L2: value (none) -> 33@100MHz
- ON: value (none) -> BLUE
- R1, R2: value (none) -> 22
- R3, R6: value (none) -> 1K
- R4: value (none) -> 330
- renumbered LED1 to ON, LED2 to L
Connections:
- net !RTS: now also IC2.!RTS; no longer IC1.!RTS
- net 3V3: now also IC1.VCC; no longer IC2.VCC
- net 5V: now also IC2.VCC; no longer IC1.VCC
- net AVCC: now also IC1.AVCC; no longer IC2.AVCC
- net D+: now also IC2.USB+; no longer IC1.USB+
- net D-: now also IC2.USB-; no longer IC1.USB-
- net FT_3V3: now also IC2.!RESET, IC2.3V3OUT, IC2.VCCIO; no longer IC1.!RESET, IC1.3V3OUT, IC1.VCCIO
- net FT_RX: now also IC1.PD7, IC2.RXD; no longer IC1.RXD, IC2.PD7
- net FT_TX: now also IC1.PD6, IC2.TXD; no longer IC1.TXD, IC2.PD6
- net PA0: now also IC1.PA0; no longer IC2.PA0
- net PA1: now also IC1.PA1; no longer IC2.PA1
- net PA2: now also IC1.PA2; no longer IC2.PA2
- net PA3: now also IC1.PA3; no longer IC2.PA3
- net PA4: now also IC1.PA4; no longer IC2.PA4
- net PA5: now also IC1.PA5; no longer IC2.PA5
- net PA6: now also IC1.PA6; no longer IC2.PA6
- net PA7: now also IC1.PA7; no longer IC2.PA7
- net PC0: now also IC1.PC0; no longer IC2.PC0
- net PC1: now also IC1.PC1; no longer IC2.PC1
- net PC2: now also IC1.PC2; no longer IC2.PC2
- net PC3: now also IC1.PC3; no longer IC2.PC3
- net PC4: now also IC1.PC4; no longer IC2.PC4
- net PC5: now also IC1.PC5; no longer IC2.PC5
- net PC6: now also IC1.PC6; no longer IC2.PC6
- net PC7: now also IC1.PC7; no longer IC2.PC7
- net PD0: now also IC1.PD0; no longer IC2.PD0
- net PD1: now also IC1.PD1; no longer IC2.PD1
- net PD2: now also IC1.PD2; no longer IC2.PD2
- net PD3: now also IC1.PD3; no longer IC2.PD3
- net PD4: now also IC1.PD4; no longer IC2.PD4
- net PD5: now also IC1.PD5; no longer IC2.PD5
- net PDI_C: now also IC1.!RESET; no longer IC2.!RESET
- net PDI_D: now also IC1.PDI; no longer IC2.PDI
- net PR0: now also IC1.PR0; no longer IC2.PR0
- net PR1: now also IC1.PR1; no longer IC2.PR1
Other:
- note removed: "v0.2"

Commit message: finished BOM
Parts:
- removed R7: (no value), Ai_Passives:RES0603
- added R5: 1K, Ai_Passives:RES0603
- R3: value 1K -> 10K
- R4: value 330 -> 300
Connections:
- net 3V3: now also R5.1; no longer R6.1
- net N$8: now also R5.2; no longer R6.2
- net N$9: now also R6.2; no longer R7.2
- net PA0: now also R6.1; no longer R7.1
Other:
- moved on the sheet: R6
Changed lines of the file:
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@@
 <part name="U1" library="Ai_Power" deviceset="MIC5219-*" device="" technology="3.3" value="MIC5219-3.3"/>
 <part name="SUPPLY5" library="Ai_Power" deviceset="GND" device=""/>
-<part name="R4" library="Ai_Passives" deviceset="RES" device="0603" value="330"/>
+<part name="R4" library="Ai_Passives" deviceset="RES" device="0603" value="300"/>
 <part name="L" library="Ai_LED" deviceset="LED" device="0603" value="YELLOW"/>
 <part name="SUPPLY6" library="Ai_Power" deviceset="GND" device=""/>
@@
 <part name="L1" library="Ai_Passives" deviceset="IND" device="0603" value="33@100MHz"/>
 <part name="L2" library="Ai_Passives" deviceset="IND" device="0603" value="33@100MHz"/>
-<part name="R3" library="Ai_Passives" deviceset="RES" device="0603" value="1K"/>
+<part name="R3" library="Ai_Passives" deviceset="RES" device="0603" value="10K"/>
 <part name="C7" library="Ai_Passives" deviceset="CAP" device="0603" value="0.1uF"/>
 <part name="C8" library="Ai_Passives" deviceset="CAP" device="0603" value="4.7uF"/>
 <part name="SUPPLY13" library="Ai_Power" deviceset="GND" device=""/>
-<part name="R6" library="Ai_Passives" deviceset="RES" device="0603" value="1K"/>
+<part name="R5" library="Ai_Passives" deviceset="RES" device="0603" value="1K"/>
 <part name="ON" library="Ai_LED" deviceset="LED" device="0603" value="BLUE"/>
 <part name="SUPPLY14" library="Ai_Power" deviceset="GND" device=""/>
 <part name="LOGO1" library="SparkFun-Aesthetics" deviceset="OSHW-LOGO" device="S"/>
-<part name="R7" library="Ai_Passives" deviceset="RES" device="0603"/>
+<part name="R6" library="Ai_Passives" deviceset="RES" device="0603" value="1K"/>
 <part name="C6" library="Ai_Passives" deviceset="CAP" device="0603" value="0.1uF"/>
 <part name="SUPPLY11" library="Ai_Power" deviceset="GND" device=""/>
@@
 <instance part="C8" gate="G$1" x="237.49" y="111.76"/>
 <instance part="SUPPLY13" gate="GND" x="229.87" y="99.06"/>
-<instance part="R6" gate="G$1" x="76.2" y="53.34" rot="MR270"/>
+<instance part="R5" gate="G$1" x="76.2" y="53.34" rot="MR270"/>
 <instance part="ON" gate="G$1" x="76.2" y="43.18"/>
 <instance part="SUPPLY14" gate="GND" x="76.2" y="33.02"/>
 <instance part="LOGO1" gate="G$1" x="132.08" y="12.7"/>
-<instance part="R7" gate="G$1" x="140.97" y="66.04" rot="R90"/>
+<instance part="R6" gate="G$1" x="140.97" y="66.04" rot="R90"/>
 <instance part="C6" gate="G$1" x="129.54" y="60.96"/>
 <instance part="SUPPLY11" gate="GND" x="129.54" y="48.26"/>
@@
 <segment>
 <wire x1="138.43" y1="58.42" x2="140.97" y2="58.42" width="0.1524" layer="91"/>
-<pinref part="R7" gate="G$1" pin="1"/>
+<pinref part="R6" gate="G$1" pin="1"/>
 <wire x1="140.97" y1="58.42" x2="144.78" y2="58.42" width="0.1524" layer="91"/>
 <wire x1="140.97" y1="60.96" x2="140.97" y2="58.42" width="0.1524" layer="91"/>
@@
 </segment>
 <segment>
-<pinref part="R6" gate="G$1" pin="1"/>
+<pinref part="R5" gate="G$1" pin="1"/>
 <pinref part="U$9" gate="G$1" pin="3V3"/>
 <wire x1="76.2" y1="58.42" x2="76.2" y2="60.96" width="0.1524" layer="91"/>
@@
 <segment>
 <pinref part="ON" gate="G$1" pin="A"/>
+<pinref part="R5" gate="G$1" pin="2"/>
+<wire x1="76.2" y1="48.26" x2="76.2" y2="45.72" width="0.1524" layer="91"/>
+</segment>
+</net>
+<net name="N$9" class="0">
+<segment>
 <pinref part="R6" gate="G$1" pin="2"/>
-<wire x1="76.2" y1="48.26" x2="76.2" y2="45.72" width="0.1524" layer="91"/>
-</segment>
-</net>
-<net name="N$9" class="0">
-<segment>
-<pinref part="R7" gate="G$1" pin="2"/>
 <wire x1="140.97" y1="71.12" x2="140.97" y2="73.66" width="0.1524" layer="91"/>
 <wire x1="140.97" y1="73.66" x2="143.51" y2="73.66" width="0.1524" layer="91"/>

Commit message: minor revision
Parts:
- LOGO1: device SparkFun-Aesthetics:OSHW-LOGOS -> Ai_Miscellany:OSHW-LOGOS
- RST: value SW-SPSTSMD03X026 -> SW-SPSTSMD035X030; device Ai_Electromechanical:SW-SPSTSMD03X026 -> Ai_Electromechanical:SW-SPSTSMD035X030
Changed lines of the file:
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@@
 <part name="ON" library="Ai_LED" deviceset="LED" device="0603" value="BLUE"/>
 <part name="SUPPLY14" library="Ai_Power" deviceset="GND" device=""/>
-<part name="LOGO1" library="SparkFun-Aesthetics" deviceset="OSHW-LOGO" device="S"/>
+<part name="LOGO1" library="Ai_Miscellany" deviceset="OSHW-LOGO" device="S"/>
 <part name="R6" library="Ai_Passives" deviceset="RES" device="0603" value="1K"/>
 <part name="C6" library="Ai_Passives" deviceset="CAP" device="0603" value="0.1uF"/>
@@
 <part name="FUSE" library="Ai_Passives" deviceset="FB" device=""/>
 <part name="USB1" library="Ai_Connectors" deviceset="USB" device="MICROB-TH" value="USBMICROB-TH"/>
-<part name="RST" library="Ai_Electromechanical" deviceset="SW-SPST" device="SMD03X026"/>
+<part name="RST" library="Ai_Electromechanical" deviceset="SW-SPST" device="SMD035X030"/>
 <part name="SUPPLY12" library="Ai_Power" deviceset="GND" device=""/>
 <part name="FRAME1" library="Ai_Miscellany" deviceset="FRAME-LETTER" device="">
